Commit message: sei la, bora pro outro

File: urdf/camera_robot.urdf (robot description, URDF)
Before this commit: robot camera_robot, 3 links, 2 joints
Joints:
- joint camera_tilt_joint: limit (none) -> lower=-1.57 upper=1.57 effort=10 velocity=1; origin xyz=0 0 0.2 rpy=0 0 0 -> xyz=0 0 3.5 rpy=0 0 0; parent head_link -> base_link; type continuous -> revolute
- joint head_yaw_joint: limit (none) -> lower=-1.57 upper=1.57 effort=10 velocity=1
