Commit message: CAMERA ROTACIONANDO DESPIROCADA, e isso eh o certo

File: urdf/camera_robot.xacro.urdf (robot description, URDF)
Before this commit: robot camera_robot, 4 links, 3 joints
Links:
- added link imu, mass 0.1
Joints:
- added joint head_to_imu: type fixed, parent head_link, child imu, origin xyz=0.0 0.0 0.0
- joint camera_tilt_joint: limit lower=-1.57 upper=1.57 effort=1000 velocity=30 -> (none); type revolute -> continuous
- joint head_yaw_joint: limit lower=-1.57 upper=1.57 effort=1000 velocity=30 -> (none); type revolute -> continuous

Commit message: consegui, coloquei 1 robo com 3 cameras posicionadas nos lugares que eu quis, se quiser adicionar mais da trabalho, se quiser alterar a fodase vc lembra tu eh foda

File: urdf/camera_robot.xacro.urdf (robot description, URDF)
Before this commit: robot camera_robot, 5 links, 4 joints
Links:
- removed link base_link
- removed link head_link
- removed link imu
- removed link neck_link
- added link base_link_0, mass 10.0; visual box size=1 1 0.5
- added link base_link_1, mass 10.0; visual box size=1 1 0.5
- added link base_link_2, mass 10.0; visual box size=1 1 0.5
- added link head_link_0, mass 1.0; visual box size=0.1 0.1 0.1
- added link head_link_1, mass 1.0; visual box size=0.1 0.1 0.1
- added link head_link_2, mass 1.0; visual box size=0.1 0.1 0.1
- added link imu_0, mass 0.1
- added link imu_1, mass 0.1
- added link imu_2, mass 0.1
- added link neck_link_0, mass 1.0; visual box size=0.1 0.1 0.1
- added link neck_link_1, mass 1.0; visual box size=0.1 0.1 0.1
- added link neck_link_2, mass 1.0; visual box size=0.1 0.1 0.1
Joints:
- removed joint camera_tilt_joint
- removed joint head_to_imu
- removed joint head_yaw_joint
- removed joint world_to_base
- added joint camera_tilt_joint_0: type continuous, parent neck_link_0, child head_link_0, origin xyz=0 0 0.3 rpy=0 0 0, axis 0 1 0
- added joint camera_tilt_joint_1: type continuous, parent neck_link_1, child head_link_1, origin xyz=0 0 0.3 rpy=0 0 0, axis 0 1 0
- added joint camera_tilt_joint_2: type continuous, parent neck_link_2, child head_link_2, origin xyz=0 0 0.3 rpy=0 0 0, axis 0 1 0
- added joint head_to_imu_0: type fixed, parent head_link_0, child imu_0, origin xyz=0.0 0.0 0.0
- added joint head_to_imu_1: type fixed, parent head_link_1, child imu_1, origin xyz=0.0 0.0 0.0
- added joint head_to_imu_2: type fixed, parent head_link_2, child imu_2, origin xyz=0.0 0.0 0.0
- added joint head_yaw_joint_0: type continuous, parent base_link_0, child neck_link_0, origin xyz=0 0 3.5 rpy=0 0 0, axis 0 0 1
- added joint head_yaw_joint_1: type continuous, parent base_link_1, child neck_link_1, origin xyz=0 0 3.5 rpy=0 0 0, axis 0 0 1
- added joint head_yaw_joint_2: type continuous, parent base_link_2, child neck_link_2, origin xyz=0 0 3.5 rpy=0 0 0, axis 0 0 1
- added joint world_to_base_0: type fixed, parent world, child base_link_0, origin xyz=-3 -7.4687 0 rpy=0 0 0
- added joint world_to_base_1: type fixed, parent world, child base_link_1, origin xyz=4.0 7.4687 0 rpy=0 0 0
- added joint world_to_base_2: type fixed, parent world, child base_link_2, origin xyz=-9.9830 -1.2500 0 rpy=0 0 0

Commit message: reposicionei as cameras

File: urdf/camera_robot.xacro.urdf (robot description, URDF)
Before this commit: robot camera_robot, 13 links, 12 joints
Joints:
- joint world_to_base_0: origin xyz=-3 -7.4687 0 rpy=0 0 0 -> xyz=-3 -7.4687 0 rpy=0 0 1.57
- joint world_to_base_1: origin xyz=4.0 7.4687 0 rpy=0 0 0 -> xyz=4.0 7.4687 0 rpy=0 0 -1.57
